Commit message: Working Depth Camera

File: baxter_description/urdf/baxter_base/baxter_base.gazebo.xacro (robot description, xacro)
@@ -58,8 +58,8 @@
   <!-- Gazebo-Specific Sensor Properties -->
   <gazebo reference="head_camera">
-    <sensor name="head_camera" type="camera">
+    <sensor name="head_camera" type="depth">
       <update_rate>30.0</update_rate>
       <camera name="head_camera">
-        <pose>0.0 0.21 0.0 0.0 -0.8 -1.570796327 </pose>
+        <pose>0.0 0.0 0.0 0.0 0.0 0.0 </pose>
         <horizontal_fov>1.3962634</horizontal_fov>
         <image>
@@ -72,23 +72,15 @@
           <far>300</far>
         </clip>
-        <noise>
-          <type>gaussian</type>
-          <mean>0.0</mean>
-          <stddev>0.007</stddev>
-        </noise>
       </camera>
-      <plugin filename="libgazebo_ros_camera.so" name="camera_controller">
-        <alwaysOn>true</alwaysOn>
-        <updateRate>0.0</updateRate>
+      <plugin filename="libgazebo_ros_openni_kinect.so" name="camera_controller">
         <cameraName>head_camera</cameraName>
         <imageTopicName>image</imageTopicName>
         <cameraInfoTopicName>camera_info</cameraInfoTopicName>
         <frameName>head_camera</frameName>
-        <hackBaseline>0.07</hackBaseline>
-        <distortionK1>0.0</distortionK1>
-        <distortionK2>0.0</distortionK2>
-        <distortionK3>0.0</distortionK3>
-        <distortionT1>0.0</distortionT1>
-        <distortionT2>0.0</distortionT2>
+            <imageTopicName>rgb/image_raw</imageTopicName>
+            <cameraInfoTopicName>rgb/camera_info</cameraInfoTopicName>
+            <depthImageTopicName>depth/image_raw</depthImageTopicName>
+            <depthImageCameraInfoTopicName>depth/camera_info</depthImageCameraInfoTopicName>
+            <pointCloudTopicName>depth/points</pointCloudTopicName>
         <robotNamespace>/cameras</robotNamespace>
       </plugin>

File: baxter_description/urdf/baxter_base/baxter_base.urdf.xacro (robot description, xacro)
@@ -229,5 +229,5 @@
   </joint>
   <joint name="head_camera" type="fixed">
-    <origin rpy="1.75057 0 1.57079632679" xyz="0.12839 0 0.06368"/>
+    <origin rpy="0 0 0" xyz="0.12839 0 0.6368"/>
     <parent link="head"/>
     <child link="head_camera"/>

Commit message: modified gripper and base urdfs

File: baxter_description/urdf/baxter_base/baxter_base.gazebo.xacro (robot description, xacro)
@@ -58,32 +58,69 @@
   <!-- Gazebo-Specific Sensor Properties -->
   <gazebo reference="head_camera">
-    <sensor name="head_camera" type="depth">
-      <update_rate>30.0</update_rate>
-      <camera name="head_camera">
-        <pose>0.0 0.0 0.0 0.0 0.0 0.0 </pose>
-        <horizontal_fov>1.3962634</horizontal_fov>
-        <image>
-          <width>800</width>
-          <height>800</height>
-          <format>R8G8B8</format>
-        </image>
-        <clip>
-          <near>0.02</near>
-          <far>300</far>
-        </clip>
-      </camera>
-      <plugin filename="libgazebo_ros_openni_kinect.so" name="camera_controller">
-        <cameraName>head_camera</cameraName>
-        <imageTopicName>image</imageTopicName>
-        <cameraInfoTopicName>camera_info</cameraInfoTopicName>
-        <frameName>head_camera</frameName>
-            <imageTopicName>rgb/image_raw</imageTopicName>
-            <cameraInfoTopicName>rgb/camera_info</cameraInfoTopicName>
-            <depthImageTopicName>depth/image_raw</depthImageTopicName>
-            <depthImageCameraInfoTopicName>depth/camera_info</depthImageCameraInfoTopicName>
-            <pointCloudTopicName>depth/points</pointCloudTopicName>
-        <robotNamespace>/cameras</robotNamespace>
-      </plugin>
-    </sensor>
+      <sensor type="depth" name="head_camera">
+        <always_on>true</always_on>
+        <update_rate>20.0</update_rate>
+        <camera>
+          <horizontal_fov>0.994</horizontal_fov>
+          <image>
+            <format>R8G8B8</format>
+            <width>640</width>
+            <height>480</height>
+          </image>
+          <clip>
+            <near>0.01</near>
+            <far>5</far>
+          </clip>
+        </camera>
+        <plugin name="camera_controller" filename="libgazebo_ros_openni_kinect.so">
+          <alwaysOn>true</alwaysOn>
+          <updateRate>20.0</updateRate>
+          <cameraName>head_camera</cameraName>
+          <imageTopicName>ir/image_raw</imageTopicName>
+          <cameraInfoTopicName>/ir/camera_info</cameraInfoTopicName>
+          <depthImageTopicName>depth/image_raw</depthImageTopicName>
+          <depthImageCameraInfoTopicName>depth/camera_info</depthImageCameraInfoTopicName>
+          <pointCloudTopicName>depth/points</pointCloudTopicName>
+          <frameName>head_camera</frameName>
+          <pointCloudCutoff>0.5</pointCloudCutoff>
+          <distortionK1>0.00000001</distortionK1>
+          <distortionK2>0.00000001</distortionK2>
+          <distortionK3>0.00000001</distortionK3>
+          <distortionT1>0.00000001</distortionT1>
+          <distortionT2>0.00000001</distortionT2>
+	  <robotNamespace>/cameras</robotNamespace>
+        </plugin>
+      </sensor>
+      <sensor type="depth" name="head_camera">
+        <always_on>true</always_on>
+        <update_rate>20.0</update_rate>
+        <camera>
+          <horizontal_fov>0.994</horizontal_fov>
+          <image>
+            <format>R8G8B8</format>
+            <width>640</width>
+            <height>480</height>
+          </image>
+          <clip>
+            <near>0.01</near>
+            <far>5</far>
+          </clip>
+        </camera>
+        <plugin name="camera_controller" filename="libgazebo_ros_openni_kinect.so">
+          <alwaysOn>true</alwaysOn>
+          <updateRate>20.0</updateRate>
+          <cameraName>head_camera</cameraName>
+          <imageTopicName>rgb/image_raw</imageTopicName>
+          <pointCloudTopicName>rgb/points</pointCloudTopicName>
+          <cameraInfoTopicName>rgb/camera_info</cameraInfoTopicName>
+          <frameName>head_camera</frameName>
+          <pointCloudCutoff>0.5</pointCloudCutoff>
+          <distortionK1>0.00000001</distortionK1>
+          <distortionK2>0.00000001</distortionK2>
+          <distortionK3>0.00000001</distortionK3>
+          <distortionT1>0.00000001</distortionT1>
+          <distortionT2>0.00000001</distortionT2>
+        </plugin>
+      </sensor>
   </gazebo>
   <gazebo reference="right_hand_camera">
@@ -94,6 +131,6 @@
         <horizontal_fov>1.3962634</horizontal_fov>
         <image>
-          <width>800</width>
-          <height>800</height>
+          <width>640</width>
+          <height>480</height>
           <format>R8G8B8</format>
         </image>

File: baxter_description/urdf/baxter_base/baxter_base.urdf.xacro (robot description, xacro)
@@ -229,5 +229,5 @@
   </joint>
   <joint name="head_camera" type="fixed">
-    <origin rpy="0 0 0" xyz="0.12839 0 0.6368"/>
+    <origin rpy="0 0.95 0" xyz="0.12839 0 0.6368"/>
     <parent link="head"/>
     <child link="head_camera"/>

File: baxter_description/urdf/left_end_effector.urdf.xacro (robot description, xacro)
@@ -4,9 +4,9 @@
   <xacro:rethink_electric_gripper side="left"
                                   l_finger="extended_narrow"
-                                  l_finger_slot="2"
+                                  l_finger_slot="3"
                                   l_finger_tip="paddle_tip"
                                   l_finger_grasp="inner"
                                   r_finger="extended_narrow"
-                                  r_finger_slot="2"
+                                  r_finger_slot="3"
                                   r_finger_tip="paddle_tip"
                                   r_finger_grasp="inner"/>
